Commit message: ADD: Joy action

File: install/cal_rtheta/share/cal_rtheta/urdf/catch.urdf (robot description, URDF)
Before this commit: robot catch, 9 links, 8 joints
Links:
- link arm2: geometry visual box size=0.05 0.05 0.2
- link body_link: geometry visual box size=0.3 0.3 0.2
- link prismatic_link: geometry visual box size=1.0 0.05 0.05
- link revolute_link: geometry visual box size=1.0 0.05 0.05
Joints:
- joint body_to_revolute: origin xyz=0 0 0.165 -> xyz=-0.5 0 0.05
- joint prismatic_to_arm2: limit lower=-0.08 upper=0.08 effort=100 velocity=0.1 -> lower=-0.04 upper=0.04 effort=100 velocity=0.1
- joint revolute_to_prismatic: limit lower=0.1 upper=0.4 effort=100 velocity=0.1 -> lower=0.25 upper=0.6 effort=100 velocity=0.1; origin xyz=0 0 0.025 rpy=0 0 0 -> xyz=0 0 0.05 rpy=0 0 0
