Commit message: ADD: enabled all  motion

File: urdf/catch.urdf (robot description, URDF)
Before this commit: robot catch, 11 links, 10 joints
Joints:
- joint arm2_to_arm3: axis (none) -> 0 0 1; limit (none) -> lower=0 upper=3.14 effort=0.5 velocity=6.0; type fixed -> revolute
- joint arm3_to_hand1: axis 0 0 1 -> (none); limit lower=-3.14 upper=3.14 effort=0.5 velocity=6.0 -> (none); type revolute -> fixed
- joint arm3_to_hand2: axis 0 0 1 -> (none); limit lower=-3.14 upper=3.14 effort=0.5 velocity=6.0 -> (none); type revolute -> fixed
- joint arm3_to_hand3: axis 0 0 1 -> (none); limit lower=-3.14 upper=3.14 effort=0.5 velocity=6.0 -> (none); type revolute -> fixed

Commit message: ADD: xy_to_rtheta

File: urdf/catch.urdf (robot description, URDF)
Before this commit: robot catch, 9 links, 8 joints
Links:
- link prismatic_link: geometry visual box size=1.0 0.05 0.025
- link revolute_link: geometry visual box size=1.0 0.05 0.025
Joints:
- joint prismatic_to_arm2: origin xyz=0.2 0 0 rpy=0 0 0 -> xyz=0.51 0 0 rpy=0 0 0
- joint revolute_to_prismatic: limit lower=0.1 upper=0.4 effort=100 velocity=0.1 -> lower=0.1 upper=0.95 effort=100 velocity=0.1

Commit message: ADD: 自動のx,yからr,theta

File: urdf/catch.urdf (robot description, URDF)
Before this commit: robot catch, 9 links, 8 joints
Links:
- link prismatic_link: geometry visual box size=0.803 0.05 0.025
- link revolute_link: geometry visual box size=0.803 0.05 0.025
Joints:
- joint prismatic_to_arm2: origin xyz=0.51 0 0 rpy=0 0 0 -> xyz=0.415 0 0 rpy=0 0 0
- joint revolute_to_prismatic: limit lower=0.1 upper=0.95 effort=100 velocity=0.1 -> lower=0.0 upper=0.542 effort=100 velocity=0.1

Commit message: ADD: ハンドの回転

File: urdf/catch.urdf (robot description, URDF)
Before this commit: robot catch, 9 links, 8 joints
Joints:
- joint arm3_to_hand1: limit lower=0 upper=3.14 effort=0.5 velocity=6.0 -> lower=-3.14 upper=3.14 effort=0.5 velocity=6.0
- joint arm3_to_hand2: limit lower=0 upper=3.14 effort=0.5 velocity=6.0 -> lower=-3.14 upper=3.14 effort=0.5 velocity=6.0
- joint arm3_to_hand3: limit lower=0 upper=3.14 effort=0.5 velocity=6.0 -> lower=-3.14 upper=3.14 effort=0.5 velocity=6.0
